Commit message: [dev]解决gazebo_ros2_control插件加载问题，新建gazebomoveit协同启动，解决虚拟关节和gazebo控制器问题

File: ur_description/urdf/test_new.urdf (robot description, URDF)
Before this commit: robot dual_arm, 52 links, 51 joints
Links:
- added link dummy_child_l_l_inner
- added link dummy_child_l_l_tip
- added link dummy_child_l_r_inner
- added link dummy_child_l_r_knuckle
- added link dummy_child_l_r_tip
- added link dummy_child_r_l_inner
- added link dummy_child_r_l_tip
- added link dummy_child_r_r_inner
- added link dummy_child_r_r_knuckle
- added link dummy_child_r_r_tip
- added link moveit_mimic_fix_dummy_root; visual box size=0.001 0.001 0.001
Joints:
- added joint left_robotiq_85_left_finger_tip_joint_mimic: type fixed, parent moveit_mimic_fix_dummy_root, child dummy_child_l_l_tip, origin xyz=0 0 0 rpy=0 0 0
- added joint left_robotiq_85_left_inner_knuckle_joint_mimic: type fixed, parent moveit_mimic_fix_dummy_root, child dummy_child_l_l_inner, origin xyz=0 0 0 rpy=0 0 0
- added joint left_robotiq_85_right_finger_tip_joint_mimic: type fixed, parent moveit_mimic_fix_dummy_root, child dummy_child_l_r_tip, origin xyz=0 0 0 rpy=0 0 0
- added joint left_robotiq_85_right_inner_knuckle_joint_mimic: type fixed, parent moveit_mimic_fix_dummy_root, child dummy_child_l_r_inner, origin xyz=0 0 0 rpy=0 0 0
- added joint left_robotiq_85_right_knuckle_joint_mimic: type fixed, parent moveit_mimic_fix_dummy_root, child dummy_child_l_r_knuckle, origin xyz=0 0 0 rpy=0 0 0
- added joint moveit_mimic_fix_to_world: type fixed, parent world, child moveit_mimic_fix_dummy_root, origin xyz=0 0 -10.0
- added joint right_robotiq_85_left_finger_tip_joint_mimic: type fixed, parent moveit_mimic_fix_dummy_root, child dummy_child_r_l_tip, origin xyz=0 0 0 rpy=0 0 0
- added joint right_robotiq_85_left_inner_knuckle_joint_mimic: type fixed, parent moveit_mimic_fix_dummy_root, child dummy_child_r_l_inner, origin xyz=0 0 0 rpy=0 0 0
- added joint right_robotiq_85_right_finger_tip_joint_mimic: type fixed, parent moveit_mimic_fix_dummy_root, child dummy_child_r_r_tip, origin xyz=0 0 0 rpy=0 0 0
- added joint right_robotiq_85_right_inner_knuckle_joint_mimic: type fixed, parent moveit_mimic_fix_dummy_root, child dummy_child_r_r_inner, origin xyz=0 0 0 rpy=0 0 0
- added joint right_robotiq_85_right_knuckle_joint_mimic: type fixed, parent moveit_mimic_fix_dummy_root, child dummy_child_r_r_knuckle, origin xyz=0 0 0 rpy=0 0 0
