Commit message: 测试附着碰撞体

File: ur_description/urdf/test.urdf (robot description, URDF)
Before this commit: robot dual_arm, 52 links, 51 joints
Links:
- added link target_plate, mass 0.2; collision box size=0.2 0.15 0.01; visual box size=0.2 0.15 0.01
Joints:
- added joint table_to_target_plate: type fixed, parent table_link, child target_plate, origin xyz=0.0 0.0 0.58 rpy=0 0 0

Commit message: 附着体读取yaml，pose tracking失败

File: ur_description/urdf/test.urdf (robot description, URDF)
Before this commit: robot dual_arm, 53 links, 52 joints
Links:
- removed link target_plate
- link left_robotiq_85_base_link: geometry collision mesh filename=package://robotiq_description/meshes/collision/2f_85/roboti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; visual mesh filename=package://robotiq_description/meshes/visual/2f_85/robotiq_b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
- link left_robotiq_85_left_finger_link: geometry collision mesh filename=package://robotiq_description/meshes/collision/2f_85/left_f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; visual mesh filename=package://robotiq_description/meshes/visual/2f_85/left_fing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
- link left_robotiq_85_left_finger_tip_link: geometry collision mesh filename=package://robotiq_description/meshes/collision/2f_85/left_f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; visual mesh filename=package://robotiq_description/meshes/visual/2f_85/left_fing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
- link left_robotiq_85_left_inner_knuckle_link: geometry collision mesh filename=package://robotiq_description/meshes/collision/2f_85/left_i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; visual mesh filename=package://robotiq_description/meshes/visual/2f_85/left_inne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
- link left_robotiq_85_left_knuckle_link: geometry collision mesh filename=package://robotiq_description/meshes/collision/2f_85/left_k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; visual mesh filename=package://robotiq_description/meshes/visual/2f_85/left_knuc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
- link left_robotiq_85_right_finger_link: geometry collision mesh filename=package://robotiq_description/meshes/collision/2f_85/right_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; visual mesh filename=package://robotiq_description/meshes/visual/2f_85/right_fin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
- link left_robotiq_85_right_finger_tip_link: geometry collision mesh filename=package://robotiq_description/meshes/collision/2f_85/right_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; visual mesh filename=package://robotiq_description/meshes/visual/2f_85/right_fin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
- link left_robotiq_85_right_inner_knuckle_link: geometry collision mesh filename=package://robotiq_description/meshes/collision/2f_85/right_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; visual mesh filename=package://robotiq_description/meshes/visual/2f_85/right_inn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
- link left_robotiq_85_right_knuckle_link: geometry collision mesh filename=package://robotiq_description/meshes/collision/2f_85/right_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; visual mesh filename=package://robotiq_description/meshes/visual/2f_85/right_knu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
- link right_robotiq_85_base_link: geometry collision mesh filename=package://robotiq_description/meshes/collision/2f_85/roboti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; visual mesh filename=package://robotiq_description/meshes/visual/2f_85/robotiq_b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
- link right_robotiq_85_left_finger_link: geometry collision mesh filename=package://robotiq_description/meshes/collision/2f_85/left_f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; visual mesh filename=package://robotiq_description/meshes/visual/2f_85/left_fing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
- link right_robotiq_85_left_finger_tip_link: geometry collision mesh filename=package://robotiq_description/meshes/collision/2f_85/left_f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; visual mesh filename=package://robotiq_description/meshes/visual/2f_85/left_fing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
- link right_robotiq_85_left_inner_knuckle_link: geometry collision mesh filename=package://robotiq_description/meshes/collision/2f_85/left_i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; visual mesh filename=package://robotiq_description/meshes/visual/2f_85/left_inne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
- link right_robotiq_85_left_knuckle_link: geometry collision mesh filename=package://robotiq_description/meshes/collision/2f_85/left_k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; visual mesh filename=package://robotiq_description/meshes/visual/2f_85/left_knuc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
- link right_robotiq_85_right_finger_link: geometry collision mesh filename=package://robotiq_description/meshes/collision/2f_85/right_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; visual mesh filename=package://robotiq_description/meshes/visual/2f_85/right_fin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
- link right_robotiq_85_right_finger_tip_link: geometry collision mesh filename=package://robotiq_description/meshes/collision/2f_85/right_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; visual mesh filename=package://robotiq_description/meshes/visual/2f_85/right_fin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
- link right_robotiq_85_right_inner_knuckle_link: geometry collision mesh filename=package://robotiq_description/meshes/collision/2f_85/right_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; visual mesh filename=package://robotiq_description/meshes/visual/2f_85/right_inn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
- link right_robotiq_85_right_knuckle_link: geometry collision mesh filename=package://robotiq_description/meshes/collision/2f_85/right_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; visual mesh filename=package://robotiq_description/meshes/visual/2f_85/right_knu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
Joints:
- removed joint table_to_target_plate

Commit message: moveit::core::RobotStatePtr和tf_buffer->lookupTransform进行末端位姿查询，解决movegroup获取不准的问题。添加moveit_visual_tools

File: ur_description/urdf/test.urdf (robot description, URDF)
Before this commit: robot dual_arm, 52 links, 51 joints
Joints:
- joint table_to_base_right: origin xyz=0.8 0.25 0.125 rpy=0 0 0 -> xyz=0.8 0.25 0.125 rpy=0 0 3.141592653589793

Commit message: [dev] ``` 初步修改 feat(motion_plan): 添加堆叠功能节点并更新依赖配置
添加了新的stack节点用于实现堆叠功能，更新了CMakeLists.txt和package.xml
以包含必要的依赖项，包括linkattacher_msgs消息包。

refactor(ur_description): 调整Gazebo仿真环境中目标物体的位置

将左右两侧目标板的位置向内移动，调整X轴坐标分别从-0.65637和0.73915
修改为-0.35637和0.43915，以改善仿真效果。

refactor(dual_ur_moveit_config): 添加双臂预堆叠姿态配置

在SRDF文件中添加了left_prestack和right_prestack两个新的组状态，
定义了双臂的预堆叠关节角度配置，并移除了过时的注释代码。

docs(README): 移除冗余标题行

删除了README.md文件中的冗余项目标题行，保持文档简洁性。
```

File: ur_description/urdf/test.urdf (robot description, URDF)
Before this commit: robot dual_arm, 52 links, 51 joints
Links:
- added link dummy_child_l_l_inner
- added link dummy_child_l_l_tip
- added link dummy_child_l_r_inner
- added link dummy_child_l_r_knuckle
- added link dummy_child_l_r_tip
- added link dummy_child_r_l_inner
- added link dummy_child_r_l_tip
- added link dummy_child_r_r_inner
- added link dummy_child_r_r_knuckle
- added link dummy_child_r_r_tip
- added link moveit_mimic_fix_dummy_root; visual box size=0.001 0.001 0.001
- link left_base_link_inertia: geometry collision mesh filename=file://$(find ur_description)/meshes/ur3e/collision/base.stl; visual mesh filename=file://$(find ur_description)/meshes/ur3e/visual/base.dae
- link left_camera_baselink: geometry collision mesh filename=file://$(find ur_description)/meshes/camera/left_camera_bas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; visual mesh filename=file://$(find ur_description)/meshes/camera/left_camera_bas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
- link left_camera_link: geometry collision mesh filename=file://$(find ur_description)/meshes/camera/left_camera_lin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; visual mesh filename=file://$(find ur_description)/meshes/camera/left_camera_lin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
- link left_forearm_link: geometry collision mesh filename=file://$(find ur_description)/meshes/ur3e/collision/forearm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; visual mesh filename=file://$(find ur_description)/meshes/ur3e/visual/forearm.dae
- link left_robotiq_85_base_link: geometry collision mesh filename=file://$(find robotiq_description)/meshes/collision/2f_85/r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; visual mesh filename=file://$(find robotiq_description)/meshes/visual/2f_85/robo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
- link left_robotiq_85_left_finger_link: geometry collision mesh filename=file://$(find robotiq_description)/meshes/collision/2f_85/l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; visual mesh filename=file://$(find robotiq_description)/meshes/visual/2f_85/left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
- link left_robotiq_85_left_finger_tip_link: geometry collision mesh filename=file://$(find robotiq_description)/meshes/collision/2f_85/l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; visual mesh filename=file://$(find robotiq_description)/meshes/visual/2f_85/left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
- link left_robotiq_85_left_inner_knuckle_link: geometry collision mesh filename=file://$(find robotiq_description)/meshes/collision/2f_85/l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; visual mesh filename=file://$(find robotiq_description)/meshes/visual/2f_85/left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
- link left_robotiq_85_left_knuckle_link: geometry collision mesh filename=file://$(find robotiq_description)/meshes/collision/2f_85/l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; visual mesh filename=file://$(find robotiq_description)/meshes/visual/2f_85/left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
- link left_robotiq_85_right_finger_link: geometry collision mesh filename=file://$(find robotiq_description)/meshes/collision/2f_85/r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; visual mesh filename=file://$(find robotiq_description)/meshes/visual/2f_85/righ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
- link left_robotiq_85_right_finger_tip_link: geometry collision mesh filename=file://$(find robotiq_description)/meshes/collision/2f_85/r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; visual mesh filename=file://$(find robotiq_description)/meshes/visual/2f_85/righ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
- link left_robotiq_85_right_inner_knuckle_link: geometry collision mesh filename=file://$(find robotiq_description)/meshes/collision/2f_85/r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; visual mesh filename=file://$(find robotiq_description)/meshes/visual/2f_85/righ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
- link left_robotiq_85_right_knuckle_link: geometry collision mesh filename=file://$(find robotiq_description)/meshes/collision/2f_85/r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; visual mesh filename=file://$(find robotiq_description)/meshes/visual/2f_85/righ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
- link left_shoulder_link: geometry collision mesh filename=file://$(find ur_description)/meshes/ur3e/collision/shoulde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; visual mesh filename=file://$(find ur_description)/meshes/ur3e/visual/shoulder.d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
- link left_upper_arm_link: geometry collision mesh filename=file://$(find ur_description)/meshes/ur3e/collision/upperar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; visual mesh filename=file://$(find ur_description)/meshes/ur3e/visual/upperarm.d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
- link left_wrist_1_link: geometry collision mesh filename=file://$(find ur_description)/meshes/ur3e/collision/wrist1.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; visual mesh filename=file://$(find ur_description)/meshes/ur3e/visual/wrist1.dae
- link left_wrist_2_link: geometry collision mesh filename=file://$(find ur_description)/meshes/ur3e/collision/wrist2.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; visual mesh filename=file://$(find ur_description)/meshes/ur3e/visual/wrist2.dae
- link left_wrist_3_link: geometry collision mesh filename=file://$(find ur_description)/meshes/ur3e/collision/wrist3.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; visual mesh filename=file://$(find ur_description)/meshes/ur3e/visual/wrist3.dae
- link right_base_link_inertia: geometry collision mesh filename=file://$(find ur_description)/meshes/ur3e/collision/base.stl; visual mesh filename=file://$(find ur_description)/meshes/ur3e/visual/base.dae
- link right_camera_baselink: geometry collision mesh filename=file://$(find ur_description)/meshes/camera/right_camera_ba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; visual mesh filename=file://$(find ur_description)/meshes/camera/right_camera_ba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
- link right_camera_link: geometry collision mesh filename=file://$(find ur_description)/meshes/camera/right_camera_li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; visual mesh filename=file://$(find ur_description)/meshes/camera/right_camera_li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
- link right_forearm_link: geometry collision mesh filename=file://$(find ur_description)/meshes/ur3e/collision/forearm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; visual mesh filename=file://$(find ur_description)/meshes/ur3e/visual/forearm.dae
- link right_robotiq_85_base_link: geometry collision mesh filename=file://$(find robotiq_description)/meshes/collision/2f_85/r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; visual mesh filename=file://$(find robotiq_description)/meshes/visual/2f_85/robo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
- link right_robotiq_85_left_finger_link: geometry collision mesh filename=file://$(find robotiq_description)/meshes/collision/2f_85/l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; visual mesh filename=file://$(find robotiq_description)/meshes/visual/2f_85/left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
- link right_robotiq_85_left_finger_tip_link: geometry collision mesh filename=file://$(find robotiq_description)/meshes/collision/2f_85/l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; visual mesh filename=file://$(find robotiq_description)/meshes/visual/2f_85/left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
- link right_robotiq_85_left_inner_knuckle_link: geometry collision mesh filename=file://$(find robotiq_description)/meshes/collision/2f_85/l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; visual mesh filename=file://$(find robotiq_description)/meshes/visual/2f_85/left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
- link right_robotiq_85_left_knuckle_link: geometry collision mesh filename=file://$(find robotiq_description)/meshes/collision/2f_85/l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; visual mesh filename=file://$(find robotiq_description)/meshes/visual/2f_85/left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
- link right_robotiq_85_right_finger_link: geometry collision mesh filename=file://$(find robotiq_description)/meshes/collision/2f_85/r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; visual mesh filename=file://$(find robotiq_description)/meshes/visual/2f_85/righ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
- link right_robotiq_85_right_finger_tip_link: geometry collision mesh filename=file://$(find robotiq_description)/meshes/collision/2f_85/r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; visual mesh filename=file://$(find robotiq_description)/meshes/visual/2f_85/righ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
- link right_robotiq_85_right_inner_knuckle_link: geometry collision mesh filename=file://$(find robotiq_description)/meshes/collision/2f_85/r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; visual mesh filename=file://$(find robotiq_description)/meshes/visual/2f_85/righ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
- link right_robotiq_85_right_knuckle_link: geometry collision mesh filename=file://$(find robotiq_description)/meshes/collision/2f_85/r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; visual mesh filename=file://$(find robotiq_description)/meshes/visual/2f_85/righ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
- link right_shoulder_link: geometry collision mesh filename=file://$(find ur_description)/meshes/ur3e/collision/shoulde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; visual mesh filename=file://$(find ur_description)/meshes/ur3e/visual/shoulder.d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
- link right_upper_arm_link: geometry collision mesh filename=file://$(find ur_description)/meshes/ur3e/collision/upperar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; visual mesh filename=file://$(find ur_description)/meshes/ur3e/visual/upperarm.d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
- link right_wrist_1_link: geometry collision mesh filename=file://$(find ur_description)/meshes/ur3e/collision/wrist1.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; visual mesh filename=file://$(find ur_description)/meshes/ur3e/visual/wrist1.dae
- link right_wrist_2_link: geometry collision mesh filename=file://$(find ur_description)/meshes/ur3e/collision/wrist2.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; visual mesh filename=file://$(find ur_description)/meshes/ur3e/visual/wrist2.dae
- link right_wrist_3_link: geometry collision mesh filename=file://$(find ur_description)/meshes/ur3e/collision/wrist3.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; visual mesh filename=file://$(find ur_description)/meshes/ur3e/visual/wrist3.dae
Joints:
- added joint left_robotiq_85_left_finger_tip_joint_mimic: type fixed, parent moveit_mimic_fix_dummy_root, child dummy_child_l_l_tip, origin xyz=0 0 0 rpy=0 0 0
- added joint left_robotiq_85_left_inner_knuckle_joint_mimic: type fixed, parent moveit_mimic_fix_dummy_root, child dummy_child_l_l_inner, origin xyz=0 0 0 rpy=0 0 0
- added joint left_robotiq_85_right_finger_tip_joint_mimic: type fixed, parent moveit_mimic_fix_dummy_root, child dummy_child_l_r_tip, origin xyz=0 0 0 rpy=0 0 0
- added joint left_robotiq_85_right_inner_knuckle_joint_mimic: type fixed, parent moveit_mimic_fix_dummy_root, child dummy_child_l_r_inner, origin xyz=0 0 0 rpy=0 0 0
- added joint left_robotiq_85_right_knuckle_joint_mimic: type fixed, parent moveit_mimic_fix_dummy_root, child dummy_child_l_r_knuckle, origin xyz=0 0 0 rpy=0 0 0
- added joint moveit_mimic_fix_to_world: type fixed, parent world, child moveit_mimic_fix_dummy_root, origin xyz=0 0 -10.0
- added joint right_robotiq_85_left_finger_tip_joint_mimic: type fixed, parent moveit_mimic_fix_dummy_root, child dummy_child_r_l_tip, origin xyz=0 0 0 rpy=0 0 0
- added joint right_robotiq_85_left_inner_knuckle_joint_mimic: type fixed, parent moveit_mimic_fix_dummy_root, child dummy_child_r_l_inner, origin xyz=0 0 0 rpy=0 0 0
- added joint right_robotiq_85_right_finger_tip_joint_mimic: type fixed, parent moveit_mimic_fix_dummy_root, child dummy_child_r_r_tip, origin xyz=0 0 0 rpy=0 0 0
- added joint right_robotiq_85_right_inner_knuckle_joint_mimic: type fixed, parent moveit_mimic_fix_dummy_root, child dummy_child_r_r_inner, origin xyz=0 0 0 rpy=0 0 0
- added joint right_robotiq_85_right_knuckle_joint_mimic: type fixed, parent moveit_mimic_fix_dummy_root, child dummy_child_r_r_knuckle, origin xyz=0 0 0 rpy=0 0 0

File: ur_description/urdf/test_new.urdf (robot description, URDF)
Before this commit: robot dual_arm, 63 links, 62 joints
Joints:
- joint table_to_base_left: origin xyz=-0.8 0.25 0.125 rpy=0 0 0 -> xyz=-0.5 0.25 0.125 rpy=0 0 0
- joint table_to_base_right: origin xyz=0.8 0.25 0.125 rpy=0 0 3.141592653589793 -> xyz=0.5 0.25 0.125 rpy=0 0 3.141592653589793
